Commit message: temp

File: robots/hydrus/ceiling_inspection.urdf.xacro (robot description, xacro)
@@ -2,4 +2,36 @@
 <robot
     xmlns:xacro="http://www.ros.org/wiki/xacro" name="hydrusx" >
-  <xacro:include filename="$(find hydrus)/robots/quad/tx2_zed_201810.urdf.xacro" />
+  <!-- basic kinematics model -->
+  <xacro:include filename="$(find hydrus)/urdf/common.xacro" />
+  <xacro:include filename="$(find hydrus)/urdf/link.urdf.xacro" />
+  <xacro:hydrusx_link self="1" child="2" rotor_direction="-1" with_battery = "0" />
+  <xacro:hydrusx_link self="2" child="3" rotor_direction="1"  with_battery = "0" />
+  <xacro:hydrusx_link self="3" child="4" rotor_direction="-1" with_battery = "0" />
+  <xacro:hydrusx_link self="4" child="4" rotor_direction="1"  with_battery = "0"/>
+  <!-- special battery arrangement -->
+  <xacro:extra_module name = "bat1" parent = "link1" visible = "1"
+                      model_url = "package://hydrus/urdf/mesh/modules/battery/Kypom-3000-6s.stl" scale="0.001">
+    <origin xyz="${link_length/2} 0.0 -0.048" rpy="${pi/2} 0 0"/>
+    <inertial>
+      <origin xyz="0 0 0" rpy="0 0 0"/>
+      <mass value="0.4108"/>
+      <inertia
+          ixx="0.0001" iyy="0.0006" izz="0.0006"
+          ixy="0.0" ixz="0.0"  iyz="0.0"/>
+    </inertial>
+  </xacro:extra_module>
+  <xacro:extra_module name = "bat2" parent = "link4" visible = "1"
+                      model_url = "package://hydrus/urdf/mesh/modules/battery/Kypom-3000-6s.stl" scale="0.001">
+    <origin xyz="${link_length/2} 0.0 -0.048" rpy="${pi/2} 0 0"/>
+    <inertial>
+      <origin xyz="0 0 0" rpy="0 0 0"/>
+      <mass value="0.4108"/>
+      <inertia
+          ixx="0.0001" iyy="0.0006" izz="0.0006"
+          ixy="0.0" ixz="0.0"  iyz="0.0"/>
+    </inertial>
+  </xacro:extra_module>
+  <!-- oboard sensors and processors -->
+  <xacro:include filename="$(find ceil_effect_control)/robots/onboards.urdf.xacro" />
+  <xacro:onboards link = "2" />
 </robot>

File: robots/onboards.urdf.xacro (robot description, xacro)
@@ -43,5 +43,5 @@
     <xacro:extra_module name = "leddarone" parent = "link${link + 1}" visible = "1"
                         model_url = "package://hydrus/urdf/mesh/modules/sensor/leddar_one_tx2_attached_mode.dae">
-      <origin xyz="0.0866 0.0 -0.06267" rpy="0 ${pi} 0"/>
+      <origin xyz="0.0866 0.0 0.03" rpy="0 0 0"/>
       <inertial>
         <origin xyz="-0.007950 0.000000 -0.000140" rpy="0 0 0"/>
