Commit message: update what?

File: robots/hydrus/robot.gazebo.xacro (robot description, xacro)
@@ -2,5 +2,8 @@
 <robot
     xmlns:xacro="http://www.ros.org/wiki/xacro" name="hydrusx" >
+  <!-- robot urdf -->
+  <xacro:include filename="$(find ceil_effect_control)/robots/hydrus/robot.urdf.xacro" />
   <!-- gazebo plugin for sensors -->
+  <!-- default sensor plugin in base model -->
   <xacro:include filename="$(find hydrus)/robots/onboards/tx2_zed_201810/onboards.gazebo.xacro" />
   <!-- upward camera for inspection -->
@@ -72,3 +75,50 @@
     </sensor>
   </gazebo>
+  <!-- tof sensor -->
+  <xacro:extra_module name = "tof" parent = "link3">
+    <origin xyz="0.0 0.0 0.015" rpy="0 ${-pi/2} 0"/>
+    <inertial>
+      <mass value = "0.00001" />
+      <origin xyz="0 0 0" rpy="0 0 0"/>
+      <inertia
+          ixx="0.000001" ixy="0.0" ixz="0.0"
+          iyy="0.000001" iyz="0.0"
+          izz="0.000002"/>
+    </inertial>
+  </xacro:extra_module>
+  <gazebo reference="tof">
+    <sensor type="ray" name="ceil_tof">
+      <pose>0 0 0 0 0 0</pose>
+      <visualize>false</visualize>
+      <update_rate>30</update_rate>
+      <ray>
+        <scan>
+          <horizontal>
+            <samples>1</samples>
+            <resolution>1</resolution>
+            <min_angle>0</min_angle>
+            <max_angle>0</max_angle>
+          </horizontal>
+        </scan>
+        <range>
+          <min>0.03</min>
+          <max>10.0</max>
+          <resolution>0.01</resolution>
+        </range>
+        <noise>
+          <type>gaussian</type>
+          <!-- Noise parameters based on published spec for Hokuyo laser
+               achieving "+-30mm" accuracy at range < 10m.  A mean of 0.0m and
+               stddev of 0.01m will put 99.7% of samples within 0.03m of the true
+               reading. -->
+          <mean>0.0</mean>
+          <stddev>0.01</stddev>
+        </noise>
+      </ray>
+      <plugin name="gazebo_ros_head_tof_controller" filename="libgazebo_ros_laser.so">
+        <topicName>/vl53l0x/range</topicName>
+        <frameName>hokuyo_link</frameName>
+      </plugin>
+    </sensor>
+  </gazebo>
 </robot>
